File: pcb-left/splotch-left.kicad_pcb (KiCad board)
At the start: 2 copper layers, 152.7 x 120.6 mm, 82 parts, among them J1 USB_C_Receptacle_USB2.0, J2 SJ-43514, J3 AVR-ISP-6, SW1 MX-NoLED, SW10 MX-NoLED, SW11 MX-NoLED, SW12 MX-NoLED, SW13 MX-NoLED, SW14 MX-NoLED, SW15 MX-NoLED, SW16 MX-NoLED, SW17 MX-NoLED, SW18 MX-NoLED, SW19 MX-NoLED, SW2 MX-NoLED, SW20 MX-NoLED, SW21 MX-NoLED, SW22 MX-NoLED, SW23 MX-NoLED, SW24 MX-NoLED, SW25 MX-NoLED, SW26 MX-NoLED, SW27 MX-NoLED, SW28 MX-NoLED, SW29 MX-NoLED, SW3 MX-NoLED, SW30 MX-NoLED, SW31 SW_Push, SW32 SW_Push, SW4 MX-NoLED, SW5 MX-NoLED, SW6 MX-NoLED, SW7 MX-NoLED, SW8 MX-NoLED, SW9 MX-NoLED, U1 ATmega328P-PU, Y1 Crystal

Commit message: v1
Parts:
- added G***: LOGO, splotch.pretty:bomb, F.Cu at (189.0, 120.1)
- added H1: MountingHole, MountingHole:MountingHole_2.2mm_M2, F.Cu at (96.8, 40.6)
- added H2: MountingHole, MountingHole:MountingHole_2.2mm_M2, F.Cu at (191.8, 44.8)
- added H3: MountingHole, MountingHole:MountingHole_2.2mm_M2, F.Cu at (213.5, 120.3)
- added H4: MountingHole, MountingHole:MountingHole_2.2mm_M2, F.Cu at (138.2, 137.7)
- added H5: MountingHole, MountingHole:MountingHole_2.2mm_M2, F.Cu at (66.3, 112.3)
- added H6: MountingHole, MountingHole:MountingHole_2.2mm_M2, F.Cu at (134.7, 76.1)
- D1, D10, D11, D12, D13, D14, D15, D16, D17, D18, D19, D2, D20, D21, D22, D23, D24, D25, D26, D27, D28, D29, D3, D30, D31, D32, D4, D5, D6, D7, D8, D9: footprint splotch.pretty:D_DO-35_SOD27_P5.08mm_Horizontal -> splotch:D_DO-35_SOD27_P5.08mm_Horizontal
- J2: footprint splotch.pretty:CUI_SJ-43514 -> splotch:CUI_SJ-43514; moved to F.Cu
- R6, SW31, SW32: moved to F.Cu
- SW1, SW10, SW11, SW12, SW14, SW15, SW16, SW17, SW18, SW2, SW20, SW21, SW22, SW23, SW24, SW25, SW27, SW28, SW29, SW3, SW30, SW4, SW5, SW6, SW8, SW9: footprint splotch.pretty:MX-1U-NoLED -> splotch:MX-1U-NoLED
- SW13, SW19: footprint splotch.pretty:MX-1.75U-NoLED -> splotch:MX-1.75U-NoLED
- SW26: footprint splotch.pretty:MX-1.25U-NoLED -> splotch:MX-1.25U-NoLED
- SW7: footprint splotch.pretty:MX-1.5U-NoLED -> splotch:MX-1.5U-NoLED
- moved J2 5.19 mm to (210.7, 45.4), turned to 180 degrees
- moved SW32 4.60 mm to (105.5, 122.1)
- moved SW31 4.60 mm to (95.9, 118.1)
- moved J1 2.18 mm to (198.4, 35.0)
- moved J3 1.52 mm to (210.1, 107.4)
Connections:
- J2 pad 2: /Serial -> /SDA
- J2 pad 3: Net-(J2-Pad3) -> /SCL
- U1 pad 2: /Serial -> Net-(U1-Pad2)
- U1 pad 27: Net-(U1-Pad27) -> /SDA
- U1 pad 28: Net-(U1-Pad28) -> /SCL
Routing:
- net /SDA: track 0.00 -> 32.3 mm
- net /Serial: track 29.2 -> 0.00 mm
- net /SCL: track 0.00 -> 24.5 mm
- net Net-(J1-PadB5): track 4.45 -> 19.0 mm
- net Net-(F1-Pad2): track 9.36 -> 22.6 mm
- net Net-(D31-Pad1): track 23.6 -> 36.6 mm
- net Net-(D32-Pad1): track 18.4 -> 26.5 mm
- net Net-(J1-PadA5): track 3.04 -> 9.51 mm
- net /Reset: track 189.7 -> 185.2 mm, vias 1 -> 0
- net /Boot: track 128.1 -> 123.7 mm
- net /MISO: track 16.1 -> 14.0 mm
- net /SCK: track 20.9 -> 18.9 mm
- net /MOSI: track 18.6 -> 17.4 mm
- net GND: vias 0 -> 3
Other:
- outline, holes or cut-outs redrawn
- board text added: "BOOT"
- board text added: "ISP"
- board text added: "L"
- board text added: "RESET"
- board text added: "hack the planet"
