File: pcb-left/splotch-left.sch (KiCad schematic (older format))
At the start: 81 parts, among them J1 USB_C_Receptacle_USB2.0, J2 SJ-43514, J3 AVR-ISP-6, SW1 MX-NoLED, SW10 MX-NoLED, SW11 MX-NoLED, SW12 MX-NoLED, SW13 MX-NoLED, SW14 MX-NoLED, SW15 MX-NoLED, SW16 MX-NoLED, SW17 MX-NoLED, SW18 MX-NoLED, SW19 MX-NoLED, SW2 MX-NoLED, SW20 MX-NoLED, SW21 MX-NoLED, SW22 MX-NoLED, SW23 MX-NoLED, SW24 MX-NoLED, SW25 MX-NoLED, SW26 MX-NoLED, SW27 MX-NoLED, SW28 MX-NoLED, SW29 MX-NoLED, SW3 MX-NoLED, SW30 MX-NoLED, SW31 SW_Push, SW32 SW_Push, SW4 MX-NoLED, SW5 MX-NoLED, SW6 MX-NoLED, SW7 MX-NoLED, SW8 MX-NoLED, SW9 MX-NoLED, U1 ATmega328P-PU, Y1 Crystal

Commit message: v1
Parts:
- added H1, H2, H3, H4, H5, H6: MountingHole, MountingHole:MountingHole_2.2mm_M2, symbol Mechanical:MountingHole
- D1, D10, D11, D12, D13, D14, D15, D16, D17, D18, D19, D2, D20, D21, D22, D23, D24, D25, D26, D27, D28, D29, D3, D30, D31, D32, D4, D5, D6, D7, D8, D9: footprint splotch.pretty:D_DO-35_SOD27_P5.08mm_Horizontal -> splotch:D_DO-35_SOD27_P5.08mm_Horizontal
- J1: symbol Connector:USB_C_Receptacle_USB2.0 -> splotch-left-rescue:USB_C_Receptacle_USB2.0-Connector
- J2: footprint splotch.pretty:CUI_SJ-43514 -> splotch:CUI_SJ-43514
- SW1, SW10, SW11, SW12, SW14, SW15, SW16, SW17, SW18, SW2, SW20, SW21, SW22, SW23, SW24, SW25, SW27, SW28, SW29, SW3, SW30, SW4, SW5, SW6, SW8, SW9: footprint splotch.pretty:MX-1U-NoLED -> splotch:MX-1U-NoLED
- SW13, SW19: footprint splotch.pretty:MX-1.75U-NoLED -> splotch:MX-1.75U-NoLED
- SW26: footprint splotch.pretty:MX-1.25U-NoLED -> splotch:MX-1.25U-NoLED
- SW7: footprint splotch.pretty:MX-1.5U-NoLED -> splotch:MX-1.5U-NoLED
Connections:
- net SDA: now reaches U1.27 (PC4)
- net SDA: now also J2.2
- net SCL: now reaches U1.28 (PC5)
- net SCL: now also J2.3
- net Serial: no longer names the net of U1.2 (PD0)
- net Serial: no longer J2.2
- no-connect marks 6 -> 4
